File: Design Files/BigClown_GPS_Teseo-LIV3F_module_v1.0.sch (EAGLE design)
At the start: 17 parts, among them IC1 TESEO-LIV3F, X1 SMA-SMD, X2 BU-SMA-H

Commit message: Add files via upload
Parts:
- added R1, R2: (no value), rcl:R-EU_M0805
Connections:
- removed net N$5: C7.2, IC1.RF_IN
- net GND: now also C7.2
- net N$2: now also IC1.RF_IN, L2.1; no longer C7.1, JP4.1
- net N$3: now also C7.1, JP4.1, L2.2; no longer JP4.2, L2.1
- net SCL: now also R2.1
- net SDA: now also R1.1
- net VCC: now also R1.2, R2.2
- net VCC_RF: now also JP4.2; no longer L2.2
Other:
- moved on the sheet: C7, JP1, JP3, JP4, L2
